Commit message: zed_camera_link

File: ros2_ws/src/my_python_package/urdf/robot.urdf.xacro (robot description, xacro)
@@ -1,12 +1,31 @@
 <?xml version="1.0"?>
 <robot xmlns:xacro="http://www.ros.org/wiki/xacro" name="my_robot">
-    <link name="base_footprint">
+     <link name="base_footprint">
+     <joint name="base_footprint_joint" type="fixed">
+        <parent link="odom"/>
+        <child link="base_footprint"/>
+        <origin xyz="0 0 0" rpy="0 0 0"/>
+    </joint>
     </link>
     <link name="base_link">
     </link>
-    <joint name="base_footprint_joint" type="fixed">
+    <joint name="base_link_joint" type="fixed">
         <parent link="base_footprint"/>
         <child link="base_link"/>
         <origin xyz="0 0 0" rpy="0 0 0"/>
     </joint>
+    <link name="laser">
+    </link>
+    <joint name="laser_joint" type="fixed">
+        <parent link="base_link"/>
+        <child link="laser"/>
+        <origin xyz="0 0 0" rpy="0 0 0"/>
+    </joint>
+    <link name="zed_camera_link">
+    </link>
+    <joint name="base_to_zed2" type="fixed">
+        <parent link="base_link" />
+        <child link="zed_camera_link" />
+        <origin xyz="0.445 0 0.4165" />
+    </joint>
 </robot>
